File: hardware/PCB Piano v1.x/audio.kicad_sch (KiCad schematic)
At the start: 24 parts, among them J3 AudioJack3_SwitchT, J8 Conn_01x02_Pin, SW2 RotaryEncoder, U11 TVL320DAC3100

Commit message: Development Phase Update
PCB layout refined more, still not complete. Trying to start a separate v1.1 PCB file to explore a 4-layer PCB.
Parts:
- removed J3: AudioJack3_SwitchT, Connector_Audio:Jack_3.5mm_CUI_SJ-3524-SMT_Horizontal, symbol Connector_Audio:AudioJack3_SwitchT
- added C26, C27: 100uF, Capacitor_SMD:C_1206_3216Metric, symbol Device:C_Polarized_Small
- added J3: AudioJack4_SwitchTR1R2S, PCBPiano_Footprints:AudioJack_TRS_Switch_TR1R2S_SJ3-35024K-SMT-TR, symbol PCB Piano Symbols:AudioJack4_SwitchTR1R2S
- R35: value 100k -> 2.2k
Connections:
- net AGND: now also J3.2 (R2)
- net HP_L: now also C26.1
- net HP_R: now also C27.1
- net HP_TS: no longer names the net of R35.2, U11.11 (VOL/MICDET)
- net HP_TS: now also J3.1 (S)
- new net: C27.2, J3.3 (R1)
- new net: C26.2, J3.8 (T)
