File: hardware/PCB Piano v1.x/led.kicad_sch (KiCad schematic)
At the start: 46 parts, among them U4 PCA9685PW, U6 PCA9685PW

Commit message: Development Phase Update
PCB layout refined more, still not complete. Trying to start a separate v1.1 PCB file to explore a 4-layer PCB.
Parts:
- removed U4, U6: PCA9685PW, Package_SO:TSSOP-28_4.4x9.7mm_P0.65mm, symbol Driver_LED:PCA9685PW
- added U4, U6: PCA9685BS, PCBPiano_Footprints:NXP_HVQFN-28_6mmx6mmx0.85mm, symbol Driver_LED:PCA9685BS
Connections:
- net +3.3V: now also U4.25 (VDD), U6.25 (VDD), U6.26 (A0)
- net GND: now also U4.1 (A3), U4.11 (VSS), U4.2 (A4), U4.20 (~{OE}), U4.21 (A5), U4.22 (EXTCLK), U4.26 (A0), U4.27 (A1), U4.28 (A2), U4.29 (VSS), U6.1 (A3), U6.11 (VSS), U6.2 (A4), U6.20 (~{OE}), U6.21 (A5), U6.22 (EXTCLK), U6.27 (A1), U6.28 (A2), U6.29 (VSS)
- net I2C1_SCL: now also U4.23 (SCL), U6.23 (SCL)
- net I2C1_SDA: now also U4.24 (SDA), U6.24 (SDA)
- net at D5.1 (K): now also U4.3 (LED0)
- net at D5.2 (A): now also RN1.4 (R4.1); no longer RN1.1 (R1.1)
- net at D13.1 (K): now also U4.12 (LED8)
- net at D20.1 (K): now also U4.19 (LED15)
- net at D8.1 (K): now also U4.6 (LED3)
- net at D8.2 (A): now also RN1.1 (R1.1); no longer RN1.4 (R4.1)
- net at D9.1 (K): now also U4.7 (LED4)
- net at D9.2 (A): now also RN2.4 (R4.1); no longer RN2.1 (R1.1)
- net at D10.1 (K): now also U4.8 (LED5)
- net at D10.2 (A): now also RN2.3 (R3.1); no longer RN2.2 (R2.1)
- net at D36.1 (K): now also U6.19 (LED15)
- net at RN1.2 (R2.1): now also D7.2 (A); no longer D6.2 (A)
- net at RN1.3 (R3.1): now also D6.2 (A); no longer D7.2 (A)
- net at D26.1 (K): now also U6.8 (LED5)
- net at D35.1 (K): now also U6.18 (LED14)
- net at D11.1 (K): now also U4.9 (LED6)
- net at D11.2 (A): now also RN2.2 (R2.1); no longer RN2.3 (R3.1)
- net at D22.1 (K): now also U6.4 (LED1)
- net at D30.1 (K): now also U6.16 (LED12)
- net at D25.1 (K): now also U6.7 (LED4)
- net at D15.1 (K): now also U4.14 (LED10)
- net at D23.1 (K): now also U6.5 (LED2)
- net at D14.1 (K): now also U4.13 (LED9)
- net at D32.1 (K): now also U6.14 (LED10)
- net at D12.2 (A): now also RN2.1 (R1.1); no longer RN2.4 (R4.1)
- net at D34.1 (K): now also U6.17 (LED13)
- net at D12.1 (K): now also U4.10 (LED7)
- net at D21.1 (K): now also U6.3 (LED0)
- net at D28.1 (K): now also U6.10 (LED7)
- net at D18.1 (K): now also U4.17 (LED13)
- net at D33.1 (K): now also U6.13 (LED9)
- net at D6.1 (K): now also U4.4 (LED1)
- net at D7.1 (K): now also U4.5 (LED2)
- net at D27.1 (K): now also U6.9 (LED6)
- net at D24.1 (K): now also U6.6 (LED3)
- net at D16.1 (K): now also U4.15 (LED11)
- net at D19.1 (K): now also U4.18 (LED14)
- net at D17.1 (K): now also U4.16 (LED12)
- net at D29.1 (K): now also U6.12 (LED8)
- net at D31.1 (K): now also U6.15 (LED11)
