File: hardware/PCB Piano v1.x/mcu.kicad_sch (KiCad schematic)
At the start: 52 parts, among them J6 Micro_SD_Card, SW3 Reset Btn, SW4 Boot Select, SW5 Octave Select, SW6 Voice Select, U1 RP2040, U2 W25Q64JVSFIM, Y1 Crystal

Commit message: Development Phase Update
PCB layout refined more, still not complete. Trying to start a separate v1.1 PCB file to explore a 4-layer PCB.
Parts:
- R17, R18, R19, R20: value 10k -> 4.7k
Other:
- moved on the sheet: C24, C25
Changed lines of the file:
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@@
 	)
 	(junction
-		(at 35.56 93.98)
+		(at 36.83 93.98)
 		(diameter 0)
 		(color 0 0 0 0)
@@
 	)
 	(junction
+		(at 71.12 81.28)
+		(diameter 0)
+		(color 0 0 0 0)
+	)
+	(junction
 		(at 133.35 20.32)
 		(diameter 0)
@@
 	)
 	(junction
-		(at 35.56 109.22)
+		(at 36.83 109.22)
 		(diameter 0)
 		(color 0 0 0 0)
@@
 	)
 	(junction
-		(at 35.56 119.38)
+		(at 36.83 119.38)
 		(diameter 0)
 		(color 0 0 0 0)
@@
 	)
 	(junction
-		(at 71.12 81.28)
-		(diameter 0)
-		(color 0 0 0 0)
-	)
-	(junction
 		(at 123.19 30.48)
 		(diameter 0)
@@
 	)
 	(junction
-		(at 35.56 81.28)
+		(at 36.83 81.28)
 		(diameter 0)
 		(color 0 0 0 0)
@@
 	(wire
 		(pts
-			(xy 35.56 81.28) (xy 35.56 93.98)
+			(xy 36.83 81.28) (xy 36.83 93.98)
 		)
 		(stroke
@@
 	(wire
 		(pts
-			(xy 35.56 93.98) (xy 35.56 96.52)
+			(xy 36.83 93.98) (xy 36.83 96.52)
 		)
 		(stroke
@@
 	(wire
 		(pts
-			(xy 35.56 78.74) (xy 35.56 81.28)
+			(xy 36.83 78.74) (xy 36.83 81.28)
 		)
 		(stroke
@@
 	(wire
 		(pts
-			(xy 35.56 109.22) (xy 26.67 109.22)
+			(xy 36.83 109.22) (xy 29.21 109.22)
 		)
 		(stroke
@@
 	(wire
 		(pts
-			(xy 35.56 119.38) (xy 35.56 121.92)
+			(xy 36.83 119.38) (xy 36.83 121.92)
 		)
 		(stroke
@@
 	(wire
 		(pts
-			(xy 35.56 109.22) (xy 44.45 109.22)
+			(xy 36.83 109.22) (xy 44.45 109.22)
 		)
 		(stroke
@@
 	(wire
 		(pts
-			(xy 26.67 93.98) (xy 35.56 93.98)
+			(xy 29.21 93.98) (xy 36.83 93.98)
 		)
 		(stroke
@@
 	(wire
 		(pts
-			(xy 35.56 81.28) (xy 71.12 81.28)
+			(xy 36.83 81.28) (xy 71.12 81.28)
 		)
 		(stroke
@@
 	(wire
 		(pts
-			(xy 35.56 109.22) (xy 35.56 119.38)
+			(xy 36.83 109.22) (xy 36.83 119.38)
 		)
 		(stroke
@@
 	(wire
 		(pts
-			(xy 35.56 119.38) (xy 66.04 119.38)
+			(xy 36.83 119.38) (xy 66.04 119.38)
 		)
 		(stroke
@@
 	(wire
 		(pts
-			(xy 26.67 93.98) (xy 26.67 96.52)
+			(xy 29.21 93.98) (xy 29.21 96.52)
 		)
 		(stroke
@@
 	(wire
 		(pts
-			(xy 26.67 101.6) (xy 26.67 109.22)
+			(xy 29.21 101.6) (xy 29.21 109.22)
 		)
 		(stroke
@@
 	(wire
 		(pts
-			(xy 35.56 93.98) (xy 44.45 93.98)
+			(xy 36.83 93.98) (xy 44.45 93.98)
 		)
 		(stroke
@@
 	(wire
 		(pts
-			(xy 35.56 101.6) (xy 35.56 109.22)
+			(xy 36.83 101.6) (xy 36.83 109.22)
 		)
 		(stroke
@@
 			)
 		)
-		(property "Value" "10k"
+		(property "Value" "4.7k"
 			(at 185.674 53.594 90)
 			(show_name no)
@@
 	(symbol
 		(lib_id "power:+3.3V")
-		(at 35.56 78.74 0)
+		(at 36.83 78.74 0)
 		(unit 1)
 		(body_style 1)
@@
 		(fields_autoplaced yes)
 		(property "Reference" "#PWR021"
-			(at 35.56 82.55 0)
+			(at 36.83 82.55 0)
 			(hide yes)
 			(show_name no)
@@
 		)
 		(property "Value" "+3.3V"
-			(at 35.56 73.66 0)
+			(at 36.83 73.66 0)
 			(show_name no)
 			(do_not_autoplace no)
@@
 		)
 		(property "Footprint" ""
-			(at 35.56 78.74 0)
+			(at 36.83 78.74 0)
 			(hide yes)
 			(show_name no)
@@
 		)
 		(property "Datasheet" ""
-			(at 35.56 78.74 0)
+			(at 36.83 78.74 0)
 			(hide yes)
 			(show_name no)
@@
 		)
 		(property "Description" "Power symbol creates a global label with name \"+3.3V\""
-			(at 35.56 78.74 0)
+			(at 36.83 78.74 0)
 			(hide yes)
 			(show_name no)
@@
 	(symbol
 		(lib_id "Device:C_Small_US")
-		(at 35.56 99.06 0)
+		(at 36.83 99.06 0)
 		(unit 1)
 		(body_style 1)
@@
 		(fields_autoplaced yes)
 		(property "Reference" "C25"
-			(at 38.1 97.9169 0)
+			(at 39.37 97.9169 0)
 			(show_name no)
 			(do_not_autoplace no)
@@
 		)
 		(property "Value" ".1uF"
-			(at 38.1 100.4569 0)
+			(at 39.37 100.4569 0)
 			(show_name no)
 			(do_not_autoplace no)
@@
 		)
 		(property "Footprint" "Capacitor_SMD:C_0603_1608Metric"
-			(at 35.56 99.06 0)
+			(at 36.83 99.06 0)
 			(hide yes)
 			(show_name no)
@@
 		)
 		(property "Datasheet" ""
-			(at 35.56 99.06 0)
+			(at 36.83 99.06 0)
 			(hide yes)
 			(show_name no)
@@
 		)
 		(property "Description" "capacitor, small US symbol"
-			(at 35.56 99.06 0)
+			(at 36.83 99.06 0)
 			(hide yes)
 			(show_name no)
@@
 			)
 		)
-		(property "Value" "10k"
+		(property "Value" "4.7k"
 			(at 195.58 53.848 90)
 			(show_name no)
@@
 			)
 		)
-		(property "Value" "10k"
+		(property "Value" "4.7k"
 			(at 200.914 53.594 90)
 			(show_name no)
@@
 			)
 		)
-		(property "Value" "10k"
+		(property "Value" "4.7k"
 			(at 190.754 53.848 90)
 			(show_name no)
@@
 	(symbol
 		(lib_id "power:GND")
-		(at 35.56 121.92 0)
+		(at 36.83 121.92 0)
 		(unit 1)
 		(body_style 1)
@@
 		(fields_autoplaced yes)
 		(property "Reference" "#PWR022"
-			(at 35.56 128.27 0)
+			(at 36.83 128.27 0)
 			(hide yes)
 			(show_name no)
@@
 		)
 		(property "Value" "GND"
-			(at 35.56 127 0)
+			(at 36.83 127 0)
 			(show_name no)
 			(do_not_autoplace no)
@@
 		)
 		(property "Footprint" ""
-			(at 35.56 121.92 0)
+			(at 36.83 121.92 0)
 			(hide yes)
 			(show_name no)
@@
 		)
 		(property "Datasheet" ""
-			(at 35.56 121.92 0)
+			(at 36.83 121.92 0)
 			(hide yes)
 			(show_name no)
@@
 		)
 		(property "Description" "Power symbol creates a global label with name \"GND\" , ground"
-			(at 35.56 121.92 0)
+			(at 36.83 121.92 0)
 			(hide yes)
 			(show_name no)
@@
 	(symbol
 		(lib_id "Device:C_Small_US")
-		(at 26.67 99.06 0)
+		(at 29.21 99.06 0)
 		(unit 1)
 		(body_style 1)
@@
 		(fields_autoplaced yes)
 		(property "Reference" "C24"
-			(at 29.21 97.9169 0)
+			(at 31.75 97.9169 0)
 			(show_name no)
 			(do_not_autoplace no)
@@
 		)
 		(property "Value" "1uF"
-			(at 29.21 100.4569 0)
+			(at 31.75 100.4569 0)
 			(show_name no)
 			(do_not_autoplace no)
@@
 		)
 		(property "Footprint" "Capacitor_SMD:C_0603_1608Metric"
-			(at 26.67 99.06 0)
+			(at 29.21 99.06 0)
 			(hide yes)
 			(show_name no)
@@
 		)
 		(property "Datasheet" ""
-			(at 26.67 99.06 0)
+			(at 29.21 99.06 0)
 			(hide yes)
 			(show_name no)
@@
 		)
 		(property "Description" "capacitor, small US symbol"
-			(at 26.67 99.06 0)
+			(at 29.21 99.06 0)
 			(hide yes)
 			(show_name no)
