File: hardware/PCB Piano v1.1/PCB Piano v1.1.kicad_pcb (KiCad board)
At the start: 2 copper layers, 280 x 110 mm, 269 parts, among them CON1 254, J1 USB_C_Receptacle_USB2.0_16P, J2 1x5 Pin Header, J3 AudioJack4_SwitchTR1R2S, J4 Conn_01x02_Pin, J5 Conn_01x02_Pin, J6 Micro_SD_Card, J7 Conn_02x10_Odd_Even, J8 Conn_01x02_Pin, SW1 MFS126D, SW2 RotaryEncoder, SW3 Reset Btn, SW4 Boot Select, SW5 Octave Select, SW6 Voice Select, U1 RP2040, U10 MTCH2120-V/SO, U11 TVL320DAC3100, U12 TLV73318PDBV, U2 74LVC1G125, U3 BQ24072RGT, U4 PCA9685BS, U5 MTCH2120-V/SO, U6 PCA9685BS, U7 W25Q128JVP, U8 TPS63001, U9 TPS61023, Y1 Crystal

Commit message: Development Phase - PCB Complete - ERC/DRC in progress
Development commit. PBC layout complete. ERC/DRC checks in progress. Swapped some connectors for JST connectors with Adafruit-style polarization.
Parts:
- removed C16: 22uF, Capacitor_Tantalum_SMD:CP_EIA-6032-20_AVX-F
- removed the C26 at (144.0, 4.45)
- removed the C27 at (144.0, 6.96)
- removed C36: .1uF, Capacitor_SMD:C_0603_1608Metric
- removed the C5 at (106.0, 12.0)
- removed the C6 at (106.0, 14.5)
- removed CON1: 254, PCBPiano_Footprints:BatteryHolder_254Clips_18650Battery
- removed J2: 1x5 Pin Header, Connector_PinHeader_2.54mm:PinHeader_1x05_P2.54mm_Vertical_SMD_Pin1Left
- removed LS1: Speaker, PCBPiano_Footprints:TestPoint_2Pads_2.5mmx2.5mm_5mmSpacing
- removed the R13 at (86.8, 51.9)
- removed R14, R36, R37: 10k, Resistor_SMD:R_0603_1608Metric
- removed SW5: Octave Select, PCBPiano_Footprints:Button_Push_KMR6
- removed SW6: Voice Select, PCBPiano_Footprints:Button_Push_KMR6
- removed TP25, TP26: TestPoint_2Pole, PCBPiano_Footprints:TestPoint_2Pads_2.5mmx2.5mm_5mmSpacing
- added C41: .1uF, Capacitor_SMD:C_0603_1608Metric, B.Cu at (93.4, 52.6)
- added C67: 10uF, Capacitor_SMD:C_0603_1608Metric, B.Cu at (273.7, 75.0)
- added J11: Speaker, Connector_JST:JST_PH_B2B-PH-SM4-TB_1x02-1MP_P2.00mm_Vertical, B.Cu at (283.7, 44.6)
- added J12: PinHeader 1x2, Connector_PinHeader_2.54mm:PinHeader_1x02_P2.54mm_Vertical_SMD_Pin1Left, B.Cu at (103.5, 53.5)
- added J9: ~, Connector_JST:JST_PH_B2B-PH-SM4-TB_1x02-1MP_P2.00mm_Vertical, B.Cu at (60.6, 36.5)
- C10, C13, C14, C15, C17, C18, C19, C20, C21, C29, C3, C4, C9, L1, L2, R1, R10, R11, R12, R13, R17, R18, R19, R2, R20, R21, R22, R23, R25, R26, R27, R28, R3, R32, R33, R34, R38, R39, R4, R40, R41, R42, R5, R6, R7, R8, R9, SW3, SW4: moved to B.Cu
- J4: value Conn_01x02_Pin -> PinHeader 1x2; moved to B.Cu
- J5: value Conn_01x02_Pin -> ~; moved to B.Cu
- J8: footprint Connector_JST:JST_SH_BM03B-SRSS-TB_1x03-1MP_P1.00mm_Vertical -> Connector_PinHeader_2.54mm:PinHeader_1x02_P2.54mm_Vertical_SMD_Pin1Left
- SW1: footprint PCBPiano_Footprints:SolderPoint_3Pads_2.54x2.54_5.08Spacing -> Connector_JST:JST_PH_B3B-PH-SM4-TB_1x03-1MP_P2.00mm_Vertical
- TPJ1, TPJ13: value Conn_01x01_Pin -> F
- TPJ10: value Conn_01x01_Pin -> D
- TPJ11: value Conn_01x01_Pin -> D# Eb
- TPJ12: value Conn_01x01_Pin -> E
- TPJ14, TPJ2: value Conn_01x01_Pin -> F# Gb
- TPJ15, TPJ3: value Conn_01x01_Pin -> G
- TPJ16, TPJ4: value Conn_01x01_Pin -> G# Ab
- TPJ17, TPJ5: value Conn_01x01_Pin -> A
- TPJ18, TPJ6: value Conn_01x01_Pin -> A# Bb
- TPJ19, TPJ7: value Conn_01x01_Pin -> B
- TPJ20, TPJ8: value Conn_01x01_Pin -> C
- TPJ9: value Conn_01x01_Pin -> C# Db
- moved J5 197.5 mm to (45.1, 41.6)
- moved J4 192.9 mm to (60.6, 58.4)
- moved SW4 129.3 mm to (72.8, 72.2)
- moved C15 116.4 mm to (56.2, 70.7), turned to 90 degrees
- moved C20 105.5 mm to (36.6, 41.0)
- moved SW3 99.3 mm to (97.1, 47.7), turned to 180 degrees
- moved R32 91.1 mm to (97.2, 45.0), turned to 180 degrees
- moved R38 90.5 mm to (78.9, 62.9)
- moved R2 89.0 mm to (104.8, 37.8), turned to -90 degrees
- moved R42 88.4 mm to (74.9, 63.7), turned to 90 degrees
- moved R39 88.1 mm to (78.9, 61.4)
- moved R23 87.7 mm to (85.5, 49.0), turned to -90 degrees
- moved R26 87.3 mm to (98.9, 52.6), turned to -90 degrees
- moved R40 85.8 mm to (78.9, 59.9)
- moved R25 85.0 mm to (97.4, 52.6), turned to -90 degrees
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- renumbered REF** to HOLE1, REF** to HOLE2, REF** to HOLE3, REF** to HOLE4, REF** to HOLE5, REF** to SWCUT
Connections:
- net /MCU/GPIO23 renamed /MCU/I2S_SDATA_MIC
- net /debug/RUN renamed /MCU/RUN
- net /debug/SWDIO renamed /MCU/SWDIO
- net Net-(CON1-POS) renamed /power/BATT_POS
- C11 pad 1: /power/CHG_OUT -> VSYS
- C12 pad 1: /power/CHG_OUT -> VSYS
- J3 pad 2: AGND -> GND
- J4 pad 1: VBUS -> GND
- J4 pad 2: GND -> VBUS
- J5 pad 1: Net-(J5-Pin_1) -> GND
- J5 pad 2: GND -> Net-(J5-Pin_2)
- J7 pad 16: GND -> /debug/CAP2_GPIO
- J7 pad 17: /debug/CAP2_GPIO -> /MCU/GPIO24
- J7 pad 18: /MCU/GPIO24 -> /MCU/GPIO19
- SW1 pad 1: Net-(J5-Pin_1) -> Net-(J5-Pin_2)
- U1 pad 30: Net-(U1-GPIO19) -> /MCU/GPIO19
- U11 pad 16: AGND -> GND
- U11 pad 20: AGND -> GND
- U11 pad 25: AGND -> GND
- U11 pad 29: AGND -> GND
- U11 pad 33: AGND -> GND
Routing:
- net +5V: track 338.4 -> 654.8 mm, vias 6 -> 10
- net +3.3V: track 444.1 -> 699.7 mm, vias 11 -> 26
- net /MCU/ENC_A: track 0.00 -> 200.0 mm, vias 0 -> 2
- net /MCU/ENC_B: track 7.05 -> 200.5 mm, vias 0 -> 2
- net /MCU/I2S_SDATA_MIC: track 2.53 -> 155.3 mm, vias 0 -> 4
- net VSYS: track 34.6 -> 171.0 mm, vias 0 -> 2
- net /MCU/USB_DP: track 22.9 -> 139.8 mm, vias 0 -> 3
- net /MCU/USB_DM: track 28.0 -> 144.8 mm, vias 0 -> 3
- net Net-(R28-Pad1): track 143.9 -> 29.2 mm
- net Net-(R30-Pad1): track 119.3 -> 5.49 mm
- net VBUS: track 91.3 -> 199.0 mm, vias 2 -> 6
- net /MCU/UART1_RX: track 21.8 -> 116.8 mm, vias 0 -> 4
- net /MCU/UART1_TX: track 18.5 -> 111.6 mm, vias 0 -> 4
- net /MCU/BOOTSEL: track 25.1 -> 116.5 mm, vias 0 -> 4
- net /MCU/I2S_SDATA: track 131.9 -> 213.7 mm, vias 0 -> 2
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- added copper zone on B.Cu, net +5V
- added copper zone on F.Cu, net +5V
- added copper zone on B.Cu, net /power/CHG_OUT
- added copper zone on F.Cu, net /power/CHG_OUT
- added copper zone on B.Cu, net GND
- added copper zone on F.Cu, net GND
- added copper zone on B.Cu, net VBUS
- added copper zone on F.Cu, net VBUS
Other:
- board text added: "+"
- board text added: "-"
- board text added: "1"
- board text added: "1.8V PS"
- board text added: "19"
- board text added: "2"
- board text added: "20"
- board text added: "3V3"
- board text added: "3V3 PS"
- board text added: "4"
- board text added: "5V"
- board text added: "5V PS"
- board text added: "8"
- board text added: "Audio Amp"
- board text added: "BATT"
- board text added: "BATT CHGR"
- board text added: "BOOTSEL"
- board text added: "CAP1_GPIO"
- board text added: "CAP2_GPIO"
- board text added: "GND"
- board text added: "GPIO19"
- board text added: "GPIO20"
- board text added: "GPIO24"
- board text added: "I2C1_SCL"
- board text added: "I2C1_SDA"
- board text added: "M"
- board text added: "O"
- board text added: "R"
- board text added: "RESET"
- board text added: "RUN/RESET"
- board text added: "STATUS LED"
- board text added: "SWCLK"
- board text added: "SWDIO"
- board text added: "TPJ TERMINALS TO CONNECT EXTERNAL TOUCH PADS (EXPERIMENT BY CONNECTING TO CONDUCTIVE OBJECTS. TURN OFF POWER BEFORE CONNECTING.)"
- board text added: "UART1_RX"
- board text added: "UART1_TX"
- board text added: "USB_DM"
- board text added: "USB_DP"
- board text added: "V"
- board text added: "VBUS"
- board text added: "VSYS"
- board text removed: "A"
- board text removed: "DOWN"
- board text removed: "E"
- board text removed: "F"
- board text removed: "G"
- board text removed: "REC"
- board text removed: "UP"
- board text removed: "VOICES"
- board text removed: "VOLUME"
- board text removed: "■■□□"

Commit message: Firmware architecture complete - PCB revision with new charger.
Firmware Architecture Complete

- Added MP2724 charger driver
- Added TLV320DAC3100 driver
- Added MTCH2120 touch driver
- Added PCA9685 driver
- Added DotStar driver
- Added rotary encoder driver
- Added touch and LED maps
- Added control/audio/voice managers
- Added audio command queue
- Added Core1 audio architecture
- Added status LED system
- Added LED animation framework

Changes hardware schematic and PCB to accommodate a newer-style USB-C sink battery charger chip and USB data MUX to protect MCU while powered off.
Parts:
- removed C10: .1uF, Capacitor_SMD:C_0603_1608Metric
- removed C11, C12: 22uF, Capacitor_Tantalum_SMD:CP_EIA-6032-20_AVX-F
- removed C9: 1uF, Capacitor_SMD:C_0603_1608Metric
- removed D37: UPWR, LED_SMD:LED_0603_1608Metric
- removed D38: CHG, LED_SMD:LED_0603_1608Metric
- removed D39: SPWR, LED_SMD:LED_0603_1608Metric
- removed J12: PinHeader 1x2, Connector_PinHeader_2.54mm:PinHeader_1x02_P2.54mm_Vertical_SMD_Pin1Left
- removed J9: ~, Connector_JST:JST_PH_B2B-PH-SM4-TB_1x02-1MP_P2.00mm_Vertical
- removed R1, R2: 5.1k, Resistor_SMD:R_0603_1608Metric
- removed R13, R8, R9: 1.5k, Resistor_SMD:R_0603_1608Metric
- removed R21, R27: 10k, Resistor_SMD:R_0603_1608Metric
- removed R3: 1.13k, Resistor_SMD:R_0603_1608Metric
- removed R4: 46.4k, Resistor_SMD:R_0603_1608Metric
- removed R5: 49.9k, Resistor_SMD:R_0603_1608Metric
- removed R6: 200k, Resistor_SMD:R_0603_1608Metric
- removed R7: 1.18k, Resistor_SMD:R_0603_1608Metric
- removed SW1: MFS126D, Connector_JST:JST_PH_B3B-PH-SM4-TB_1x03-1MP_P2.00mm_Vertical
- removed SWCUT: MFS126D, PCBPiano_Footprints:Switch_Slide_MFS126E_PanelCutout
- removed TPJ1, TPJ13: F, PCBPiano_Footprints:Terminal_SMD_.250in
- removed TPJ10: D, PCBPiano_Footprints:Terminal_SMD_.250in
- removed TPJ11: D# Eb, PCBPiano_Footprints:Terminal_SMD_.250in
- removed TPJ12: E, PCBPiano_Footprints:Terminal_SMD_.250in
- removed TPJ14, TPJ2: F# Gb, PCBPiano_Footprints:Terminal_SMD_.250in
- removed TPJ15, TPJ3: G, PCBPiano_Footprints:Terminal_SMD_.250in
- removed TPJ16, TPJ4: G# Ab, PCBPiano_Footprints:Terminal_SMD_.250in
- removed TPJ17, TPJ5: A, PCBPiano_Footprints:Terminal_SMD_.250in
- removed TPJ18, TPJ6: A# Bb, PCBPiano_Footprints:Terminal_SMD_.250in
- removed TPJ19, TPJ7: B, PCBPiano_Footprints:Terminal_SMD_.250in
- removed TPJ20, TPJ8: C, PCBPiano_Footprints:Terminal_SMD_.250in
- removed TPJ9: C# Db, PCBPiano_Footprints:Terminal_SMD_.250in
- removed U3: BQ24072RGT, Package_DFN_QFN:VQFN-16-1EP_3x3mm_P0.5mm_EP1.6x1.6mm
- added C36: 220pF, Capacitor_SMD:C_0603_1608Metric, B.Cu at (35.9, 42.5)
- added C42: 47uF, Capacitor_Tantalum_SMD:CP_EIA-3528-15_AVX-H, B.Cu at (41.0, 39.2)
- added C68: .1uF, Capacitor_SMD:C_0603_1608Metric, B.Cu at (55.4, 61.8)
- added C69: .1uF, Capacitor_SMD:C_0603_1608Metric, B.Cu at (31.8, 78.8)
- added C70: .1uF, Capacitor_SMD:C_0603_1608Metric, B.Cu at (95.2, 40.3)
- added C74: 1uF, Capacitor_SMD:C_0603_1608Metric, B.Cu at (66.8, 46.9)
- added C75: 22nF, Capacitor_SMD:C_0603_1608Metric, B.Cu at (64.1, 55.0)
- added C77: 10uF, Capacitor_SMD:C_0805_2012Metric, B.Cu at (67.7, 49.7)
- added C78: 47uF, Capacitor_Tantalum_SMD:CP_EIA-3528-15_AVX-H, B.Cu at (44.2, 53.7)
- added C79: 47uF, Capacitor_Tantalum_SMD:CP_EIA-3528-15_AVX-H, B.Cu at (44.2, 48.5)
- added C80: 10uF, Capacitor_SMD:C_0805_2012Metric, B.Cu at (57.6, 46.9)
- added C81: 10uF, Capacitor_SMD:C_0805_2012Metric, B.Cu at (57.6, 48.9)
- added C82: 10uF, Capacitor_SMD:C_0805_2012Metric, B.Cu at (63.3, 44.4)
- added C83: 10uF, Capacitor_SMD:C_0805_2012Metric, B.Cu at (57.6, 50.9)
- added C84: 10uF, Capacitor_SMD:C_0805_2012Metric, B.Cu at (57.6, 52.9)
- added D41: APA102-2020, PCBPiano_Footprints:APA102-2020, F.Cu at (31.5, 84.0)
- added D43: LTST-C191TBKT, PCBPiano_Footprints:LED_0603_1608Metric, F.Cu at (44.5, 37.0)
- added D44: LTST-C191TBKT, PCBPiano_Footprints:LED_0603_1608Metric, F.Cu at (55.5, 37.0)
- added D45: LTST-C191TBKT, PCBPiano_Footprints:LED_0603_1608Metric, F.Cu at (93.0, 37.0)
- added J2: JST PH 4-PIN, Connector_JST:JST_PH_B4B-PH-SM4-TB_1x04-1MP_P2.00mm_Vertical, B.Cu at (58.8, 37.4)
- added JP1: SolderJumper_2_Open, Jumper:SolderJumper-2_P1.3mm_Open_RoundedPad1.0x1.5mm, B.Cu at (104.2, 44.2)
- added JP2: SolderJumper_2_Open, Jumper:SolderJumper-2_P1.3mm_Open_RoundedPad1.0x1.5mm, B.Cu at (104.2, 41.3)
- added L3: 1uH, PCBPiano_Footprints:L_Sumida_0530CDMCCDS-1R0MC_5.4x5.2mm, B.Cu at (67.7, 54.0)
- added R14: 100k, Resistor_SMD:R_0603_1608Metric, B.Cu at (40.0, 44.9)
- added R36: 100k, Resistor_SMD:R_0603_1608Metric, B.Cu at (102.2, 52.6)
- added R37: 100k, Resistor_SMD:R_0603_1608Metric, B.Cu at (94.4, 41.9)
- added R69: 100k, Resistor_SMD:R_0603_1608Metric, B.Cu at (95.1, 37.6)
- added R70: 100k, Resistor_SMD:R_0603_1608Metric, B.Cu at (67.9, 68.8)
- added R71: 100k, Resistor_SMD:R_0603_1608Metric, B.Cu at (55.4, 65.7)
- added R72: 100k, Resistor_SMD:R_0603_1608Metric, B.Cu at (59.5, 68.3)
- added R75: 1.5k, Resistor_SMD:R_0603_1608Metric, B.Cu at (47.7, 42.2)
- added R76: 1.5k, Resistor_SMD:R_0603_1608Metric, B.Cu at (47.7, 43.8)
- added R77: 1.5k, Resistor_SMD:R_0603_1608Metric, B.Cu at (47.7, 45.4)
- added R78: 10k, Resistor_SMD:R_0603_1608Metric, B.Cu at (61.9, 55.0)
- added SP1: ~, PCBPiano_Footprints:Pad_Solder_SMT_5x7mm, B.Cu at (37.5, 115.8)
- added SP10: ~, PCBPiano_Footprints:Pad_Solder_SMT_5x7mm, B.Cu at (152.5, 115.8)
- added SP11: ~, PCBPiano_Footprints:Pad_Solder_SMT_5x7mm, B.Cu at (164.0, 92.3)
- added SP12: ~, PCBPiano_Footprints:Pad_Solder_SMT_5x7mm, B.Cu at (175.5, 115.9)
- added SP13: ~, PCBPiano_Footprints:Pad_Solder_SMT_5x7mm, B.Cu at (198.5, 115.8)
- added SP14: ~, PCBPiano_Footprints:Pad_Solder_SMT_5x7mm, B.Cu at (210.1, 92.3)
- added SP15: ~, PCBPiano_Footprints:Pad_Solder_SMT_5x7mm, B.Cu at (221.5, 115.8)
- added SP16: ~, PCBPiano_Footprints:Pad_Solder_SMT_5x7mm, B.Cu at (233.0, 92.3)
- added SP17: ~, PCBPiano_Footprints:Pad_Solder_SMT_5x7mm, B.Cu at (244.5, 115.8)
- added SP18: ~, PCBPiano_Footprints:Pad_Solder_SMT_5x7mm, B.Cu at (256.0, 92.3)
- added SP19: ~, PCBPiano_Footprints:Pad_Solder_SMT_5x7mm, B.Cu at (267.5, 115.8)
- added SP2: ~, PCBPiano_Footprints:Pad_Solder_SMT_5x7mm, B.Cu at (49.0, 92.3)
- added SP20: ~, PCBPiano_Footprints:Pad_Solder_SMT_5x7mm, B.Cu at (290.5, 115.8)
- added SP3: ~, PCBPiano_Footprints:Pad_Solder_SMT_5x7mm, B.Cu at (60.5, 115.8)
- added SP4: ~, PCBPiano_Footprints:Pad_Solder_SMT_5x7mm, B.Cu at (72.0, 92.3)
- added SP5: ~, PCBPiano_Footprints:Pad_Solder_SMT_5x7mm, B.Cu at (83.5, 115.8)
- added SP6: ~, PCBPiano_Footprints:Pad_Solder_SMT_5x7mm, B.Cu at (95.0, 92.3)
- added SP7: ~, PCBPiano_Footprints:Pad_Solder_SMT_5x7mm, B.Cu at (106.5, 115.8)
- added SP8: ~, PCBPiano_Footprints:Pad_Solder_SMT_5x7mm, B.Cu at (129.5, 115.8)
- added SP9: ~, PCBPiano_Footprints:Pad_Solder_SMT_5x7mm, B.Cu at (141.0, 92.3)
- added SW5: JST-PH 1x03 SMT, Connector_JST:JST_PH_B3B-PH-SM4-TB_1x03-1MP_P2.00mm_Vertical, B.Cu at (51.0, 52.2)
- added SWCUT1: ~, PCBPiano_Footprints:Switch_Slide_MFS126E_PanelCutout, F.Cu at (77.5, 37.0)
- added TP25: TestPoint_Square, PCBPiano_Footprints:TestPoint_Pad_1.0x1.0mm, B.Cu at (61.3, 45.3)
- added U14: PI3USB102G, PCBPiano_Footprints:TQFN-10_ZL_1.6x1.3mm_P0.4mm, B.Cu at (98.6, 41.4)
- added U15: MP2724GRH-0000-P, PCBPiano_Footprints:QFN-22_2.5x3.2mm_P0.4mm, B.Cu at (63.0, 49.5)
- C1, C15, C2, C20, C21, C60, C62: value 22uF -> 47uF; footprint Capacitor_Tantalum_SMD:CP_EIA-6032-20_AVX-F -> Capacitor_Tantalum_SMD:CP_EIA-3528-15_AVX-H
- C49, C52, C54, C56, C58, C67: footprint Capacitor_SMD:C_0603_1608Metric -> Capacitor_SMD:C_0805_2012Metric
- C63: value .1uF -> 10uF; footprint Capacitor_SMD:C_0603_1608Metric -> Capacitor_SMD:C_0805_2012Metric
- D1, D2, D3, D4: value ~ -> ESD321; footprint Diode_SMD:D_SOD-523 -> PCBPiano_Footprints:D_SOD-523
- D10: value A#0 -> LTST-C191TBKT; footprint LED_SMD:LED_0603_1608Metric -> PCBPiano_Footprints:LED_0603_1608Metric
- D11: value B0 -> LTST-C191TBKT; footprint LED_SMD:LED_0603_1608Metric -> PCBPiano_Footprints:LED_0603_1608Metric
- D12: value C1 -> LTST-C191TBKT; footprint LED_SMD:LED_0603_1608Metric -> PCBPiano_Footprints:LED_0603_1608Metric
- D13: value C#1 -> LTST-C191TBKT; footprint LED_SMD:LED_0603_1608Metric -> PCBPiano_Footprints:LED_0603_1608Metric
- D14: value D1 -> LTST-C191TBKT; footprint LED_SMD:LED_0603_1608Metric -> PCBPiano_Footprints:LED_0603_1608Metric
- D15: value D#1 -> LTST-C191TBKT; footprint LED_SMD:LED_0603_1608Metric -> PCBPiano_Footprints:LED_0603_1608Metric
- D16: value E1 -> LTST-C191TBKT; footprint LED_SMD:LED_0603_1608Metric -> PCBPiano_Footprints:LED_0603_1608Metric
- D17: value F1 -> LTST-C191TBKT; footprint LED_SMD:LED_0603_1608Metric -> PCBPiano_Footprints:LED_0603_1608Metric
- D18: value F#1 -> LTST-C191TBKT; footprint LED_SMD:LED_0603_1608Metric -> PCBPiano_Footprints:LED_0603_1608Metric
- D19: value G1 -> LTST-C191TBKT; footprint LED_SMD:LED_0603_1608Metric -> PCBPiano_Footprints:LED_0603_1608Metric
- D20: value G#1 -> LTST-C191TBKT; footprint LED_SMD:LED_0603_1608Metric -> PCBPiano_Footprints:LED_0603_1608Metric
- D21: value A1 -> LTST-C191TBKT; footprint LED_SMD:LED_0603_1608Metric -> PCBPiano_Footprints:LED_0603_1608Metric
- D22: value A1# -> LTST-C191TBKT; footprint LED_SMD:LED_0603_1608Metric -> PCBPiano_Footprints:LED_0603_1608Metric
- D23: value B1 -> LTST-C191TBKT; footprint LED_SMD:LED_0603_1608Metric -> PCBPiano_Footprints:LED_0603_1608Metric
- D24: value C2 -> LTST-C191TBKT; footprint LED_SMD:LED_0603_1608Metric -> PCBPiano_Footprints:LED_0603_1608Metric
- D25: value OS-2 -> LTST-C191TBKT; footprint LED_SMD:LED_0603_1608Metric -> PCBPiano_Footprints:LED_0603_1608Metric
- D26: value OS-1 -> LTST-C191TBKT; footprint LED_SMD:LED_0603_1608Metric -> PCBPiano_Footprints:LED_0603_1608Metric
- D27: value OS0 -> LTST-C191TBKT; footprint LED_SMD:LED_0603_1608Metric -> PCBPiano_Footprints:LED_0603_1608Metric
- D28: value OS+1 -> LTST-C191TBKT; footprint LED_SMD:LED_0603_1608Metric -> PCBPiano_Footprints:LED_0603_1608Metric
- D29: value OS+2 -> LTST-C191TBKT; footprint LED_SMD:LED_0603_1608Metric -> PCBPiano_Footprints:LED_0603_1608Metric
- D30: value VS3 -> LTST-C191TBKT; footprint LED_SMD:LED_0603_1608Metric -> PCBPiano_Footprints:LED_0603_1608Metric
- D31: value VS2 -> LTST-C191TBKT; footprint LED_SMD:LED_0603_1608Metric -> PCBPiano_Footprints:LED_0603_1608Metric
- D32: value VS1 -> LTST-C191TBKT; footprint LED_SMD:LED_0603_1608Metric -> PCBPiano_Footprints:LED_0603_1608Metric
- D33: value VS0 -> LTST-C191TBKT; footprint LED_SMD:LED_0603_1608Metric -> PCBPiano_Footprints:LED_0603_1608Metric
- D34: value MIDI -> LTST-C191TBKT; footprint LED_SMD:LED_0603_1608Metric -> PCBPiano_Footprints:LED_0603_1608Metric
- D35: value LEFT -> LTST-C191TBKT; footprint LED_SMD:LED_0603_1608Metric -> PCBPiano_Footprints:LED_0603_1608Metric
- D36: value RIGHT -> LTST-C191TBKT; footprint LED_SMD:LED_0603_1608Metric -> PCBPiano_Footprints:LED_0603_1608Metric
- D40: value APA102 -> APA102-2020; footprint LED_SMD:LED_RGB_5050-6 -> PCBPiano_Footprints:APA102-2020
- D5: value F0 -> LTST-C191TBKT; footprint LED_SMD:LED_0603_1608Metric -> PCBPiano_Footprints:LED_0603_1608Metric
- D6: value F#0 -> LTST-C191TBKT; footprint LED_SMD:LED_0603_1608Metric -> PCBPiano_Footprints:LED_0603_1608Metric
- D7: value G0 -> LTST-C191TBKT; footprint LED_SMD:LED_0603_1608Metric -> PCBPiano_Footprints:LED_0603_1608Metric
- D8: value G#0 -> LTST-C191TBKT; footprint LED_SMD:LED_0603_1608Metric -> PCBPiano_Footprints:LED_0603_1608Metric
- D9: value A0 -> LTST-C191TBKT; footprint LED_SMD:LED_0603_1608Metric -> PCBPiano_Footprints:LED_0603_1608Metric
- H1: renamed from HOLE1; value MountingHole_3.2mm_M3 -> MountingHole
- H2: renamed from HOLE2; value MountingHole_3.2mm_M3 -> MountingHole
- H3: renamed from HOLE3; value MountingHole_3.2mm_M3 -> MountingHole
- H4: renamed from HOLE4; value MountingHole_3.2mm_M3 -> MountingHole
- H5: renamed from HOLE5; value MountingHole_3.2mm_M3 -> MountingHole
- J1: value USB_C_Receptacle_USB2.0_16P -> USB4110-GF-A; footprint Connector_USB:USB_C_Receptacle_GCT_USB4110 -> PCBPiano_Footprints:USB_C_Receptacle_GCT_USB4110
- J11: value Speaker -> JST-PH 1x02 SMT
- J3: value AudioJack4_SwitchTR1R2S -> SJ3-35024K-SMT-TR
- J4: value PinHeader 1x2 -> PinHeader 1x02 SMT
- J5: value ~ -> PinHeader 1x02 SMT
- J6: value Micro_SD_Card -> DM3D-SF; footprint Connector_Card:microSD_HC_Hirose_DM3D-SF -> PCBPiano_Footprints:microSD_HC_Hirose_DM3D-SF
- J7: value Conn_02x10_Odd_Even -> PinHeader 2x10 SMT Odd_Even
- J8: value Conn_01x02_Pin -> PinHeader 1x02 SMT
- L1: footprint Inductor_SMD:L_1008_2520Metric -> PCBPiano_Footprints:L_Bourns_SRP4020T_4.06x4.45x2.0mm
- L2: footprint Inductor_SMD:L_1008_2520Metric -> PCBPiano_Footprints:L_Pulse_BMRB00060630_7.3x6.6mm
- R26: value 10k -> 100k
- R68: value 2.2k -> 100k
- RN1, RN2, RN3, RN4, RN5, RN6, RN7, RN8: footprint Resistor_SMD:R_Array_Convex_4x1206 -> PCBPiano_Footprints:R_Array_Convex_4x1206
- SW2: value RotaryEncoder -> SWT0115-020025SSA_REVA; footprint PCBPiano_Footprints:Switch_RotaryEncoder_MER1045-24 -> PCBPiano_Footprints:SW_SWT0115-020025SSA_REVA
- SW3: value Reset Btn -> SWT0115-020025SSA_REVA; footprint PCBPiano_Footprints:Button_Push_KMR6 -> PCBPiano_Footprints:SW_SWT0115-020025SSA_REVA
- SW4: value Boot Select -> MER1045-24; footprint PCBPiano_Footprints:Button_Push_KMR6 -> PCBPiano_Footprints:Switch_RotaryEncoder_MER1045-24
- TP1, TP13: value F -> ~
- TP10: value D -> ~
- TP11: value D# EЬ -> ~
- TP12: value E -> ~
- TP14, TP2: value F# GЬ -> ~
- TP15, TP3: value G -> ~
- TP16, TP4: value G# AЬ -> ~
- TP17, TP5: value A -> ~
- TP18, TP6: value A# BЬ -> ~
- TP19, TP7: value B -> ~
- TP20, TP8: value C -> ~
- TP21: value OS -> ~
- TP22: value VS -> ~
- TP23: value MODE -> ~
- TP24: value AUX -> ~
- TP9: value C# DЬ -> ~
- U10, U5: value MTCH2120-V/SO -> MTCH2120-V/REB; footprint Package_SO:SOIC-20W_7.5x12.8mm_P1.27mm -> Package_DFN_QFN:VQFN-20-1EP_3x3mm_P0.4mm_EP1.7x1.7mm
- U2: value 74LVC1G125 -> 74AHCT125; footprint Package_TO_SOT_SMD:SOT-353_SC-70-5 -> Package_DFN_QFN:DHVQFN-14-1EP_2.5x3mm_P0.5mm_EP1x1.5mm
- U8: footprint Package_SON:Texas_DRC0010J_ThermalVias -> PCBPiano_Footprints:Texas_DRC0010J
- Y1: value Crystal -> FC3BSHFEM12.0-T3
- moved SW4 213.6 mm to (286.0, 86.0), turned to 180 degrees
- moved SW2 192.7 mm to (97.1, 47.7), turned to 0 degrees
- moved C63 38.8 mm to (34.1, 43.0), turned to 90 degrees
- moved SW3 33.8 mm to (74.1, 72.5)
- moved J4 18.3 mm to (73.0, 44.9), turned to -90 degrees
- moved C1 10.8 mm to (73.5, 50.5), turned to 0 degrees
- moved R22 10.2 mm to (83.6, 49.0)
- moved C4 9.16 mm to (118.7, 77.4), turned to 0 degrees
- moved C7 8.08 mm to (117.8, 97.2), turned to 180 degrees
- moved U4 8.00 mm to (118.0, 83.0)
- moved U6 8.00 mm to (187.0, 83.0)
- moved C5 7.70 mm to (187.8, 77.7)
- moved C6 7.70 mm to (187.8, 76.0)
- moved C3 6.92 mm to (118.7, 75.7), turned to 0 degrees
- moved C20 6.89 mm to (41.0, 35.7)
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Connections:
- net Net-(D1-K) renamed /power/USB_CC1
- net Net-(D2-K) renamed /power/USB_CC2
- C63 pad 1: +3.3V -> +5V
- C64 pad 1: +3.3V -> +5V
- D3 pad 1: /MCU/USB_DP -> /power/USB_DM
- D4 pad 1: /MCU/USB_DM -> /power/USB_DP
- D40 pad 1: /MCU/SPI0_MOSI -> Net-(D40-CKO)
- D40 pad 2: Net-(D40-CI) -> +5V
- D40 pad 3: GND -> Net-(D40-CKI)
- D40 pad 4: +3.3V -> Net-(D40-SDO)
- D40 pad 5: unconnected-(D40-CO-Pad5) -> GND
- D40 pad 6: unconnected-(D40-DO-Pad6) -> Net-(D40-SDI)
- J1 pad A6: /MCU/USB_DP -> /power/USB_DM
- J1 pad A7: /MCU/USB_DM -> /power/USB_DP
- J1 pad B6: /MCU/USB_DP -> /power/USB_DM
- J1 pad B7: /MCU/USB_DM -> /power/USB_DP
- J6 pad 10: (no net) -> unconnected-(J6-DET_A-Pad10)
- J6 pad 9: (no net) -> unconnected-(J6-DET_B-Pad9)
- J7 pad 10: /MCU/USB_DM -> /debug/DEBUG_DM
- J7 pad 18: /MCU/GPIO19 -> GND
- J7 pad 9: /MCU/USB_DP -> /debug/DEBUG_DP
- R15 pad 2: /MCU/USB_DP -> /MCU/MCU_DM
- R16 pad 2: /MCU/USB_DM -> /MCU/MCU_DP
- R22 pad 1: /MCU/CHG_EN2 -> /MCU/CHG_~{INT}
- R26 pad 2: /MCU/DS_ENABLE -> /MCU/DS_~{EN}
- R67 pad 1: Net-(D40-CI) -> Net-(D40-SDI)
- SW2 pad 1: (no net) -> GND
- SW3 pad 2: /MCU/RUN -> GND
- SW3 pad 3: (no net) -> /MCU/BOOTSEL
- SW3 pad 4: (no net) -> unconnected-(SW3-Pad4)
- U1 pad 13: /MCU/CHG_~{CE} -> /MCU/USB_SEL
- U1 pad 14: /MCU/CHG_EN1 -> unconnected-(U1-GPIO11-Pad14)
- U1 pad 15: /MCU/CHG_EN2 -> unconnected-(U1-GPIO12-Pad15)
- U1 pad 16: /MCU/CHG_~{PG} -> unconnected-(U1-GPIO13-Pad16)
- U1 pad 17: /MCU/CHG_~{CHG} -> /MCU/CHG_~{INT}
- U1 pad 29: /MCU/DS_ENABLE -> /MCU/DS_~{EN}
- U1 pad 30: /MCU/GPIO19 -> /MCU/5V_EN
- U1 pad 31: Net-(J12-Pin_1) -> /LED/LED_~{EN}
- U10 pad 1: +3.3V -> /MCU/I2C0_SCL
- U10 pad 10: Net-(U10-BUTTON6) -> Net-(U10-BUTTON5)
- U10 pad 11: Net-(U10-BUTTON7) -> /MCU/CAP2_~{INT}
- U10 pad 12: Net-(U10-BUTTON8) -> /debug/CAP2_GPIO
- U10 pad 13: Net-(U10-BUTTON9) -> Net-(U10-BUTTON6)
- U10 pad 14: Net-(U10-BUTTON10) -> Net-(U10-BUTTON7)
- U10 pad 15: Net-(U10-BUTTON11) -> Net-(U10-BUTTON8)
- U10 pad 16: /MCU/CAPx_~{RST} -> Net-(U10-BUTTON9)
- U10 pad 17: /MCU/I2C0_SDA -> Net-(U10-BUTTON10)
- U10 pad 18: /MCU/I2C0_SCL -> Net-(U10-BUTTON11)
- U10 pad 19: GND -> /MCU/CAPx_~{RST}
- U10 pad 2: Net-(U10-BUTTON0) -> GND
- U10 pad 20: GND -> /MCU/I2C0_SDA
- U10 pad 3: Net-(U10-BUTTON1) -> GND
- U10 pad 4: Net-(U10-BUTTON2) -> +3.3V
- U10 pad 5: Net-(U10-BUTTON3) -> Net-(U10-BUTTON0)
- U10 pad 6: Net-(U10-BUTTON4) -> Net-(U10-BUTTON1)
- U10 pad 7: Net-(U10-BUTTON5) -> Net-(U10-BUTTON2)
- U10 pad 8: /MCU/CAP2_~{INT} -> Net-(U10-BUTTON3)
- U10 pad 9: /debug/CAP2_GPIO -> Net-(U10-BUTTON4)
- U2 pad 1: /MCU/DS_ENABLE -> /MCU/DS_~{EN}
- U2 pad 2: /MCU/SPI0_SCK -> /MCU/SPI0_MOSI
- U2 pad 3: GND -> Net-(D40-SDI)
- U2 pad 4: Net-(D40-CI) -> /MCU/DS_~{EN}
- U2 pad 5: +3.3V -> /MCU/SPI0_SCK
- U4 pad 20: GND -> /LED/LED_~{EN}
- U5 pad 1: +3.3V -> /MCU/I2C0_SCL
- U5 pad 10: Net-(U5-BUTTON6) -> Net-(U5-BUTTON5)
- U5 pad 11: Net-(U5-BUTTON7) -> /MCU/CAP1_~{INT}
- U5 pad 12: Net-(U5-BUTTON8) -> /debug/CAP1_GPIO
- U5 pad 13: Net-(U5-BUTTON9) -> Net-(U5-BUTTON6)
- U5 pad 14: Net-(U5-BUTTON10) -> Net-(U5-BUTTON7)
- U5 pad 15: Net-(U5-BUTTON11) -> Net-(U5-BUTTON8)
- U5 pad 16: /MCU/CAPx_~{RST} -> Net-(U5-BUTTON9)
- U5 pad 17: /MCU/I2C0_SDA -> Net-(U5-BUTTON10)
- U5 pad 18: /MCU/I2C0_SCL -> Net-(U5-BUTTON11)
- U5 pad 19: GND -> /MCU/CAPx_~{RST}
- U5 pad 2: Net-(U5-BUTTON0) -> GND
- U5 pad 20: GND -> /MCU/I2C0_SDA
- U5 pad 3: Net-(U5-BUTTON1) -> GND
- U5 pad 4: Net-(U5-BUTTON2) -> +3.3V
- U5 pad 5: Net-(U5-BUTTON3) -> Net-(U5-BUTTON0)
- U5 pad 6: Net-(U5-BUTTON4) -> Net-(U5-BUTTON1)
- U5 pad 7: Net-(U5-BUTTON5) -> Net-(U5-BUTTON2)
- U5 pad 8: /MCU/CAP1_~{INT} -> Net-(U5-BUTTON3)
- U5 pad 9: /debug/CAP1_GPIO -> Net-(U5-BUTTON4)
- U6 pad 20: GND -> /LED/LED_~{EN}
- U9 pad 2: VSYS -> /MCU/5V_EN
- Y1 pad 2: Net-(C39-Pad1) -> GND
- Y1 pad 3: (no net) -> Net-(C39-Pad1)
- Y1 pad 4: (no net) -> GND
Routing:
- net /MCU/USB_DM: track 144.8 -> 0.00 mm, vias 3 -> 0
- net /LED/LED_~{EN}: track 0.00 -> 144.5 mm, vias 0 -> 4
- net /MCU/USB_DP: track 139.8 -> 0.00 mm, vias 3 -> 0
- net /MCU/5V_EN: track 0.00 -> 94.1 mm, vias 0 -> 4
- net /MCU/DS_ENABLE: track 79.5 -> 0.00 mm, vias 4 -> 0
- net /MCU/DS_~{EN}: track 0.00 -> 78.3 mm, vias 0 -> 5
- net VBUS: track 199.0 -> 120.9 mm, vias 6 -> 2
- net /debug/DEBUG_DM: track 0.00 -> 72.9 mm
- net /MCU/GPIO19: track 70.3 -> 0.00 mm, vias 2 -> 0
- net /MCU/CHG_~{PG}: track 67.7 -> 0.00 mm, vias 2 -> 0
- net /debug/DEBUG_DP: track 0.00 -> 64.2 mm
- net /MCU/CHG_~{CHG}: track 59.5 -> 0.00 mm, vias 2 -> 0
- net Net-(D45-A): track 0.00 -> 57.3 mm, vias 0 -> 1
- net GND: track 69.6 -> 13.5 mm
- net /MCU/MCU_DP: track 0.00 -> 55.7 mm, vias 0 -> 2
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- added copper zone on B.Cu, net /power/battery charger 2/BATT_POS
- added copper zone on B.Cu, net /power/battery charger 2/CHG_OUT
- added copper zone on B.Cu, net Net-(U15B-SW)
- added copper zone on B.Cu, net Net-(U8-L1)
- added copper zone on B.Cu, net Net-(U8-L2)
- added copper zone on B.Cu, net Net-(U9-SW)
- added copper zone on B.Cu, net VSYS
- removed copper zone on F.Cu, net +5V
- removed copper zone on B.Cu, net /power/CHG_OUT
- removed copper zone on F.Cu, net /power/CHG_OUT
- removed copper zone on F.Cu, net VBUS
Other:
- board text added: "(EXPERIMENT BY CONNECTING TO CONDUCTIVE OBJECTS. TURN OFF POWER BEFORE CONNECTING.)"
- board text added: "*J5 ACTIVE ONLY WHEN POWER OFF"
- board text added: "MCU"
- board text added: "MCU STATUS"
- board text added: "SP* SOLDER PADS. POPULATE WITH FAVORITE QUICK CONNECT TERMINALS."
- board text added: "SPKR"
- board text added: "STATUS"
- board text added: "USB POWER IN: 5V 2A"
- board text added: "VSYS*"
- board text removed: "BATT"
- board text removed: "BATT CHGR"
- board text removed: "GPIO19"
- board text removed: "GPIO20"
- board text removed: "STATUS LED"
- board text removed: "TPJ TERMINALS TO CONNECT EXTERNAL TOUCH PADS (EXPERIMENT BY CONNECTING TO CONDUCTIVE OBJECTS. TURN OFF POWER BEFORE CONNECTING.)"

Commit message: PCB Finalized and Ordered. Firmware near completion.
PCB Finalized and Ordered. Final revisions included fixing bugs on some peripheral chips. Also added an RTC circuit after realizing the SD card could benefit from adding file timestamps.

Firmware near completion. Still need to finalize some SD card operations. Synth audio core is finished and all the board peripheral chip drivers were completed.
Parts:
- removed U15: MP2724GRH-0000-P, PCBPiano_Footprints:QFN-22_2.5x3.2mm_P0.4mm
- added C71: .1uF, Capacitor_SMD:C_0603_1608Metric, B.Cu at (109.8, 74.7)
- added D37: Schottky, Diode_SMD:D_SOD-123, B.Cu at (112.6, 72.8)
- added FID1: Fiducial, Fiducial:Fiducial_1mm_Mask3mm, B.Cu at (288.5, 30.5)
- added FID2: Fiducial, Fiducial:Fiducial_1mm_Mask3mm, B.Cu at (131.0, 30.5)
- added FID3: Fiducial, Fiducial:Fiducial_1mm_Mask3mm, B.Cu at (28.5, 107.0)
- added Q1: P-Ch Power MOSFET, PCBPiano_Footprints:PPAK_3x3, B.Cu at (56.5, 44.0)
- added R27: 100k, Resistor_SMD:R_0603_1608Metric, B.Cu at (70.8, 60.0)
- added R73: 100k, Resistor_SMD:R_0603_1608Metric, B.Cu at (122.2, 97.5)
- added R74: 100k, Resistor_SMD:R_0603_1608Metric, B.Cu at (185.9, 87.6)
- added R79: 100k, Resistor_SMD:R_0603_1608Metric, B.Cu at (54.6, 47.5)
- added U13: USB C Sink Ctrl/Batt Chgr, PCBPiano_Footprints:QFN-22_2.5x3.2mm_P0.4mm, B.Cu at (63.0, 49.5)
- added U3: RTC, Package_DFN_QFN:DFN-10-1EP_2.6x2.6mm_P0.5mm_EP1.3x2.2mm, B.Cu at (109.3, 72.2)
- added Y2: 32.768kHz, PCBPiano_Footprints:Crystal_Kyocera_DT32_3.2x1.5mm, B.Cu at (105.4, 72.1)
- C1: footprint Capacitor_Tantalum_SMD:CP_EIA-3528-15_AVX-H -> Capacitor_Tantalum_SMD:CP_EIA-7343-43_Kemet-X
- C2: value 47uF -> 1F; footprint Capacitor_Tantalum_SMD:CP_EIA-3528-15_AVX-H -> PCBPiano_Footprints:SuperCap_HType_FoldedOutLegs
- C75: footprint Capacitor_SMD:C_0603_1608Metric -> Capacitor_SMD:C_0805_2012Metric
- D10, D11, D12, D13, D14, D15, D16, D17, D18, D19, D20, D21, D22, D23, D24, D25, D26, D27, D28, D29, D30, D31, D32, D33, D34, D35, D36, D43, D44, D45, D5, D6, D7, D8, D9: value LTST-C191TBKT -> 3.3fV 180mcd
- D40, D41: value APA102-2020 -> Dotstar LED
- J11: value JST-PH 1x02 SMT -> JST-PH 2-PIN SMT
- J3: value SJ3-35024K-SMT-TR -> 3.5mm TRRS
- J4, J5, J8: footprint Connector_PinHeader_2.54mm:PinHeader_1x02_P2.54mm_Vertical_SMD_Pin1Left -> Connector_PinHeader_2.54mm:PinHeader_1x02_P2.54mm_Vertical_SMD_Pin1Right
- J6: value DM3D-SF -> micro SD Card Slot
- JP1, JP2: footprint Jumper:SolderJumper-2_P1.3mm_Open_RoundedPad1.0x1.5mm -> PCBPiano_Footprints:SolderJumper-2_P1.3mm_Open_RoundedPad1.0x1.5mm
- MK1: value ICS-43432 -> MEMS I2S Microphone
- R25: value 10k -> 100k
- R43, R44, R45, R46, R47, R48, R49, R50, R51, R52, R53, R54, R55, R56, R57, R58, R59, R60, R61, R62, R63, R64, R65, R66: value 1k -> 10k
- R68: value 100k -> 10k
- R71: value 100k -> 150; footprint Resistor_SMD:R_0603_1608Metric -> Resistor_SMD:R_1206_3216Metric
- R72: value 100k -> 1k
- SW2, SW3: value SWT0115-020025SSA_REVA -> Pushbutton MO
- SWCUT1: value ~ -> MFS 126 D
- U10, U5: value MTCH2120-V/REB -> Touch Controller
- U11: value TVL320DAC3100 -> Audio DAC Class-D I2S/I2C
- U12: value TLV73318PDBV -> 1.8V
- U14: value PI3USB102G -> 1:2 USB MUX
- U2: value 74AHCT125 -> Dual Line Buffer; footprint Package_DFN_QFN:DHVQFN-14-1EP_2.5x3mm_P0.5mm_EP1x1.5mm -> Package_SO:VSSOP-8_2.3x2mm_P0.5mm
- U4, U6: value PCA9685BS -> LED Controller
- U7: value W25Q128JVP -> 128MBit
- U8: value TPS63001 -> 3.3V
- U9: value TPS61023 -> 5V
- Y1: value FC3BSHFEM12.0-T3 -> 12MHz
- moved C2 132.4 mm to (205.7, 62.0), turned to 90 degrees
- moved R71 60.0 mm to (115.0, 72.8), turned to -90 degrees
- moved R72 17.8 mm to (76.4, 73.9), turned to 180 degrees
- moved R22 3.26 mm to (83.0, 45.8), turned to 180 degrees
- moved C1 2.60 mm to (73.5, 53.1), turned to -90 degrees
- moved SW3 2.08 mm to (72.9, 70.8)
- moved C23 1.87 mm to (98.2, 67.1)
- moved U2 1.58 mm to (60.0, 62.5)
- moved C43 1.30 mm to (96.7, 67.1)
- moved C54 1.20 mm to (288.5, 70.0)
- moved C53 1.20 mm to (286.6, 69.7)
- moved C48 0.97 mm to (285.0, 69.7)
- moved C49 0.80 mm to (283.1, 70.0)
- moved C78 0.60 mm to (44.2, 54.3)
- moved SW1 0.60 mm to (51.0, 52.8)
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- renumbered SW5 to SW1
Connections:
- net /MCU/SPI0_CS renamed /MCU/SPI0_~{CS}
- net Net-(D10-K) renamed /LED/LED_105
- net Net-(D11-K) renamed /LED/LED_106
- net Net-(D12-K) renamed /LED/LED_107
- net Net-(D13-K) renamed /LED/LED_108
- net Net-(D14-K) renamed /LED/LED_109
- net Net-(D15-K) renamed /LED/LED_110
- net Net-(D16-K) renamed /LED/LED_204
- net Net-(D17-K) renamed /LED/LED_205
- net Net-(D18-K) renamed /LED/LED_206
- net Net-(D19-K) renamed /LED/LED_207
- net Net-(D20-K) renamed /LED/LED_208
- net Net-(D21-K) renamed /LED/LED_209
- net Net-(D22-K) renamed /LED/LED_210
- net Net-(D23-K) renamed /LED/LED_211
- net Net-(D24-K) renamed /LED/LED_212
- net Net-(D25-K) renamed /LED/LED_115
- net Net-(D26-K) renamed /LED/LED_114
- net Net-(D27-K) renamed /LED/LED_113
- net Net-(D28-K) renamed /LED/LED_112
- net Net-(D29-K) renamed /LED/LED_111
- net Net-(D30-K) renamed /LED/LED_200
- net Net-(D31-K) renamed /LED/LED_201
- net Net-(D32-K) renamed /LED/LED_202
- net Net-(D33-K) renamed /LED/LED_203
- net Net-(D34-K) renamed /LED/LED_215
- net Net-(D35-K) renamed /LED/LED_214
- net Net-(D36-K) renamed /LED/LED_213
- net Net-(D5-K) renamed /LED/LED_100
- net Net-(D6-K) renamed /LED/LED_101
- net Net-(D7-K) renamed /LED/LED_102
- net Net-(D8-K) renamed /LED/LED_103
- net Net-(D9-K) renamed /LED/LED_104
- net Net-(J2-Pin_3) renamed /power/battery charger 2/TH1_POS
- net Net-(R43-Pad2) renamed /touch/TOUCH_100
- net Net-(R44-Pad2) renamed /touch/TOUCH_101
- net Net-(R45-Pad2) renamed /touch/TOUCH_102
- net Net-(R46-Pad2) renamed /touch/TOUCH_103
- net Net-(R47-Pad2) renamed /touch/TOUCH_104
- net Net-(R48-Pad2) renamed /touch/TOUCH_105
- net Net-(R49-Pad2) renamed /touch/TOUCH_106
- net Net-(R50-Pad2) renamed /touch/TOUCH_107
- net Net-(R51-Pad2) renamed /touch/TOUCH_108
- net Net-(R52-Pad2) renamed /touch/TOUCH_109
- net Net-(R53-Pad2) renamed /touch/TOUCH_110
- net Net-(R54-Pad2) renamed /touch/TOUCH_111
- net Net-(R55-Pad2) renamed /touch/TOUCH_200
- net Net-(R56-Pad2) renamed /touch/TOUCH_201
- net Net-(R57-Pad2) renamed /touch/TOUCH_202
- net Net-(R58-Pad2) renamed /touch/TOUCH_203
- net Net-(R59-Pad2) renamed /touch/TOUCH_204
- net Net-(R60-Pad2) renamed /touch/TOUCH_205
- net Net-(R61-Pad2) renamed /touch/TOUCH_206
- net Net-(R62-Pad2) renamed /touch/TOUCH_207
- net Net-(R63-Pad2) renamed /touch/TOUCH_208
- net Net-(R64-Pad2) renamed /touch/TOUCH_209
- net Net-(R65-Pad2) renamed /touch/TOUCH_210
- net Net-(R66-Pad2) renamed /touch/TOUCH_211
- C2 pad 1: VBUS -> /MCU/RTC_BATT
- C80 pad 1: /power/battery charger 2/BATT_POS -> /power/battery charger 2/CHG_BATT
- C81 pad 1: /power/battery charger 2/BATT_POS -> /power/battery charger 2/CHG_BATT
- J6 pad 10: unconnected-(J6-DET_A-Pad10) -> /MCU/SD_DET
- J6 pad 9: unconnected-(J6-DET_B-Pad9) -> GND
- J7 pad 18: GND -> /MCU/GPIO11
- JP1 pad 1: /power/USB_DP -> /debug/DEBUG_DP
- JP1 pad 2: /debug/DEBUG_DP -> /power/USB_DP
- JP2 pad 1: /power/USB_DM -> /debug/DEBUG_DM
- JP2 pad 2: /debug/DEBUG_DM -> /power/USB_DM
- R22 pad 1: /MCU/CHG_~{INT} -> +3.3V
- R22 pad 2: GND -> /MCU/CHG_~{INT}
- R34 pad 2: /MCU/BOOTSEL -> Net-(U1-~{QSPI_SS})
- R71 pad 1: +3.3V -> /MCU/RTC_BATT
- R71 pad 2: Net-(R71-Pad2) -> /MCU/RTC_VDD
- R72 pad 1: Net-(R72-Pad1) -> Net-(U1-~{QSPI_SS})
- R72 pad 2: GND -> /MCU/BOOTSEL
- U1 pad 11: /MCU/UART1_TX -> /MCU/SD_DET
- U1 pad 12: /MCU/UART1_RX -> /MCU/CHG_~{INT}
- U1 pad 14: unconnected-(U1-GPIO11-Pad14) -> /MCU/GPIO11
- U1 pad 15: unconnected-(U1-GPIO12-Pad15) -> /MCU/UART1_TX
- U1 pad 16: unconnected-(U1-GPIO13-Pad16) -> /MCU/UART1_RX
- U1 pad 17: /MCU/CHG_~{INT} -> unconnected-(U1-GPIO14-Pad17)
- U1 pad 56: /MCU/BOOTSEL -> Net-(U1-~{QSPI_SS})
- U10 pad 2: GND -> Net-(U10-ADD_SEL)
- U2 pad 2: /MCU/SPI0_MOSI -> /MCU/SPI0_SCK
- U2 pad 4: /MCU/DS_~{EN} -> GND
- U2 pad 5: /MCU/SPI0_SCK -> /MCU/SPI0_MOSI
- U2 pad 7: GND -> /MCU/DS_~{EN}
- U2 pad 8: unconnected-(U2-Pad8) -> +5V
- U5 pad 2: GND -> Net-(U5-ADD_SEL)
- U7 pad 1: /MCU/BOOTSEL -> Net-(U1-~{QSPI_SS})
Routing:
- net /MCU/RTC_BATT: track 0.00 -> 97.6 mm
- net /MCU/GPIO11: track 0.00 -> 80.6 mm, vias 0 -> 2
- net /MCU/SD_DET: track 0.00 -> 65.7 mm, vias 0 -> 4
- net /power/battery charger 2/CHG_OUT: track 17.1 -> 81.9 mm, vias 2 -> 4
- net +3.3V: track 705.5 -> 670.0 mm, vias 28 -> 37
- net Net-(U1-~{QSPI_SS}): track 0.00 -> 25.2 mm
- net /MCU/BOOTSEL: track 115.7 -> 91.4 mm
- net /MCU/DS_~{EN}: track 78.3 -> 64.9 mm, vias 5 -> 6
- net /power/battery charger 2/CHG_VCC: track 43.2 -> 55.4 mm
- net /LED/I2C1_SDA: track 333.5 -> 343.8 mm, vias 8 -> 9
- net /MCU/RTC_VDD: track 0.00 -> 8.90 mm
- net /LED/I2C1_SCL: track 340.4 -> 347.9 mm, vias 8 -> 9
- net Net-(R72-Pad1): track 6.78 -> 0.00 mm, vias 2 -> 0
- net Net-(R71-Pad2): track 6.35 -> 0.00 mm
- net /power/battery charger 2/CHG_BATT: track 0.00 -> 6.22 mm, vias 0 -> 2
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- added copper zone on B.Cu, net +3.3V
- added copper zone on F.Cu, net +3.3V
- added copper zone on B.Cu, net /power/battery charger 2/CHG_BATT
- added copper zone on B.Cu, net Net-(U13B-PMID)
- added copper zone on F.Cu, net VBUS
Other:
- board text added: "!J5 ACTIVE ONLY WHEN POWER OFF"
- board text added: "!VSYS"
- board text added: "(RTC&C2 OPTIONAL)"
- board text added: "*USB_DM"
- board text added: "G"
- board text added: "GPIO11"
- board text added: "RTC"
- board text added: "SUPERCAP FOR RTC (DNP IF RTC NOT POP'D)"
- board text added: "TH"
- board text added: "USB_DP*"
- board text removed: "*J5 ACTIVE ONLY WHEN POWER OFF"
- board text removed: "USB_DM"
- board text removed: "USB_DP"
- board text removed: "VSYS*"
